File: Hardware/Food_Dispenser_Control/Food_Dispenser_Control.kicad_sch (KiCad schematic)
At the start: 71 parts, among them J1 Motor Output, J2 USB_C_Receptacle_USB2.0_16P, J3 Conn_01x02_Pin, J5 Conn_01x01, J6 Conn_01x01, J7 Conn_01x04_Pin, J8 Motor Output, J9 Motor Output, SW1 CK_KMS2xxG, SW2 SW_Push, SW3 CK_KMS2xxG, U1 ESP32-C3-MINI-1, U2 AP2112K-3.3, U3 TPS61022, U4 MCP73871, U5 DRV8833PW, U6 DRV8833PW, U7 HX711, U8 DRV8833PW

Commit message: s3 migration
Parts:
- added J10: Conn_01x03_Pin, symbol Connector:Conn_01x03_Pin
- added J4: Conn_01x07_Pin, symbol Connector:Conn_01x07_Pin
- added R26, R29: 10KOhms, Resistor_SMD:R_0805_2012Metric_Pad1.20x1.40mm_HandSolder, symbol Device:R
- added R27, R28: 22Ohms, Resistor_SMD:R_0805_2012Metric_Pad1.20x1.40mm_HandSolder, symbol Device:R
- added SW4, SW5: CK_KMS2xxG, Button_Switch_SMD:SW_SPST_CK_KMS2xxG, symbol Switch:CK_KMS2xxG
- added U9: ESP32-S3-WROOM-1, PCM_Espressif:ESP32-S3-WROOM-1, symbol PCM_Espressif:ESP32-S3-WROOM-1
Connections:
- net +3.3V: now also J4.1 (Pin_1), R26.1, R29.1
- net D+: now also R27.2
- net D-: now also R28.1
- net GND: now also J4.7 (Pin_7), SW4.2, SW4.SH (B), SW5.2, SW5.SH (B), U9.1 (GND), U9.40 (GND), U9.41 (GND)
- new net: R26.2, SW4.1, U9.3 (EN)
- new net: R27.1, U9.14 (GPIO20/U1CTS/ADC2_CH9/CLK_OUT1/USB_D+)
- new net: R28.2, U9.13 (GPIO19/U1RTS/ADC2_CH8/CLK_OUT2/USB_D-)
- new net: R29.2, SW5.1, U9.27 (GPIO0/BOOT)
- new net GPIO1_1: J10.1 (Pin_1)
- new net GPIO1_2: J10.2 (Pin_2)
- new net GPIO1_3: J10.3 (Pin_3)
- new net SCL: J4.3 (Pin_3)
- new net SDA: J4.2 (Pin_2)
- new net XSHUT1: J4.4 (Pin_4)
- new net XSHUT2: J4.5 (Pin_5)
- new net XSHUT3: J4.6 (Pin_6)
Other:
- note added: "Battery Charger/Monitor"
- note added: "Battery Input"
- note added: "IR Sensor Bus"
- note added: "IR Sensor Bus 2"
- note added: "Load Cell Ac to Dc Amp"
- note added: "Load Cell Connector"
- note added: "Motor Controllers"
- note added: "USB C Receptacle"
- moved on the sheet: C10, C11, C12, C13, C14, C15, C16, C17, C18, C19, C20, C21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

Commit message: schematic and footprints
Parts:
- removed C3: 0.1uF, Capacitor_SMD:C_0805_2012Metric_Pad1.18x1.45mm_HandSolder, symbol Device:C_Small
- removed C4: 10uF, Capacitor_SMD:C_0805_2012Metric_Pad1.18x1.45mm_HandSolder, symbol Device:C_Small
- removed R1, R11, R12, R5, R9: 10KOhms, Resistor_SMD:R_0805_2012Metric_Pad1.20x1.40mm_HandSolder, symbol Device:R
- removed R7, R8: 22Ohms, Resistor_SMD:R_0805_2012Metric_Pad1.20x1.40mm_HandSolder, symbol Device:R
- removed SW1, SW3, SW4, SW5: CK_KMS2xxG, Button_Switch_SMD:SW_SPST_CK_KMS2xxG, symbol Switch:CK_KMS2xxG
- removed U1: ESP32-C3-MINI-1, PCM_Espressif:ESP32-C3-MINI-1, symbol PCM_Espressif:ESP32-C3-MINI-1
- added C25: 0.1uF, Capacitor_SMD:C_0805_2012Metric_Pad1.18x1.45mm_HandSolder, symbol Device:C_Small
- added C26: 10uF, Capacitor_SMD:C_0805_2012Metric_Pad1.18x1.45mm_HandSolder, symbol Device:C_Small
- added R30: 10KOhms, Resistor_SMD:R_0805_2012Metric_Pad1.20x1.40mm_HandSolder, symbol Device:R
- added SW1, SW6: SW_Push, Button_Switch_THT:SW_PUSH_6mm_H5mm, symbol Switch:SW_Push
- J1, J7, J8, J9: footprint Connector_JST:JST_XH_B4B-XH-AM_1x04_P2.50mm_Vertical -> TerminalBlock_Phoenix:TerminalBlock_Phoenix_MKDS-1,5-4_1x04_P5.00mm_Horizontal
- J10: footprint (none) -> TerminalBlock_Phoenix:TerminalBlock_Phoenix_MKDS-1,5-3_1x03_P5.00mm_Horizontal
- J3: footprint Connector_JST:JST_PH_S2B-PH-K_1x02_P2.00mm_Horizontal -> TerminalBlock_Phoenix:TerminalBlock_Phoenix_MKDS-1,5-2_1x02_P5.00mm_Horizontal
- J4: footprint (none) -> TerminalBlock_Phoenix:TerminalBlock_Phoenix_MKDS-1,5-7_1x07_P5.00mm_Horizontal
- SW2: footprint Button_Switch_SMD:SW_SPST_PTS645 -> Button_Switch_THT:SW_PUSH_6mm_H5mm
Connections:
- net +3.3V: now also U9.2 (3V3), C25.2, C26.2, R30.2
- net DIRA: now also U9.17 (GPIO9/TOUCH9/ADC1_CH8/FSPIHD/SUBSPIHD)
- net DIRB: now also U9.7 (GPIO7/TOUCH7/ADC1_CH6)
- net DOUT: now also U9.19 (GPIO11/TOUCH11/ADC2_CH0/FSPID/FSPIIO5/SUBSPID)
- net EN1: now also U9.4 (GPIO4/TOUCH4/ADC1_CH3)
- net EN2: now also U9.5 (GPIO5/TOUCH5/ADC1_CH4)
- net EN3: now also U9.6 (GPIO6/TOUCH6/ADC1_CH5)
- net GND: now also C25.1, C26.1, SW1.1, SW6.2
- net GPIO1_1: now also U9.31 (GPIO38/FSPIWP/SUBSPIWP)
- net GPIO1_2: now also U9.26 (GPIO45)
- net GPIO1_3: now also U9.16 (GPIO46)
- net PD_SCK: now also U9.20 (GPIO12/TOUCH12/ADC2_CH1/FSPICLK/FSPIIO6/SUBSPICLK)
- net PERC: now also U9.38 (GPIO2/TOUCH2/ADC1_CH1)
- net PWMA: now also U9.18 (GPIO10/TOUCH10/ADC1_CH9/FSPICS0/FSPIIO4/SUBSPICS0)
- net PWMB: now also U9.12 (GPIO8/TOUCH8/ADC1_CH7/SUBSPICS1)
- net SCL: now also U9.22 (GPIO14/TOUCH14/ADC2_CH3/FSPIWP/FSPIDQS/SUBSPIWP)
- net SDA: now also U9.21 (GPIO13/TOUCH13/ADC2_CH2/FSPIQ/FSPIIO7/SUBSPIQ)
- net STAT: now also U9.39 (GPIO1/TOUCH1/ADC1_CH0)
- net Sleep: now also U9.15 (GPIO3/TOUCH3/ADC1_CH2), R30.1, SW6.1; no longer SW2.1
- net XSHUT1: now also U9.10 (GPIO17/U1TXD/ADC2_CH6)
- net XSHUT2: now also U9.11 (GPIO18/U1RXD/ADC2_CH7/CLK_OUT3)
- net XSHUT3: now also U9.23 (GPIO21)
- net at R26.2, U9.3 (EN): now also SW2.1
- net at R29.2, U9.27 (GPIO0/BOOT): now also SW1.2
- no-connect marks 9 -> 8
Other:
- note added: "Microcontroller"
- note added: "Status LED's"
- note added: "Voltage Regulators"
- moved on the sheet: C1, C2, C5, C6, D1, L1, R10, R2, R26, R27, R28, R29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

Commit message: Some stuff idk
Parts:
- removed C2, C6: 1uF, Capacitor_SMD:C_0805_2012Metric_Pad1.18x1.45mm_HandSolder, symbol Device:C_Small
- removed L1: 1u, Inductor_SMD:L_0805_2012Metric_Pad1.15x1.40mm_HandSolder, symbol Device:L
- removed R4: 100k, Resistor_SMD:R_0805_2012Metric_Pad1.20x1.40mm_HandSolder, symbol Device:R
- removed U3: TPS61022, Package_DFN_QFN:Texas_RWU0007A_VQFN-7_2x2mm_P0.5mm, symbol Converter_DCDC:TPS61022
- added C3: 10uF, Capacitor_SMD:C_0805_2012Metric_Pad1.18x1.45mm_HandSolder, symbol Device:C_Small
- added D3: LED, LED_SMD:LED_0805_2012Metric_Pad1.15x1.40mm_HandSolder, symbol Device:LED
- added R1: 22Ohms, Resistor_SMD:R_0805_2012Metric_Pad1.20x1.40mm_HandSolder, symbol Device:R
- added SW3: SW_SPST, symbol Switch:SW_SPST
- added U1: MCP73831-2-OT, Package_TO_SOT_SMD:SOT-23-5, symbol Battery_Management:MCP73831-2-OT
- R3: value 732k -> 2KOhms
Connections:
- net +5.0V: no longer C11.2, C12.2, C16.2, C17.2, C23.2, C24.2, R3.2, U5.12 (VM), U6.12 (VM), U8.12 (VM)
- net GND: now also R3.1, C3.1, U1.2 (V_{SS})
- net VBAT: now also SW3.1 (A), U1.3 (V_{BAT})
- net VBUS: now also C3.2, D3.2 (A), U1.4 (V_{DD})
- net VOUT: no longer C1.2, U2.1 (VIN), U2.3 (EN)
- new net: R3.2, U1.5 (PROG)
- new net: D3.1 (K), R1.1
- new net: R1.2, U1.1 (STAT)
- new net VBAT_SYS: C1.2, C11.2, C12.2, C16.2, C17.2, C23.2, C24.2, SW3.2 (B), U2.1 (VIN), U2.3 (EN), U5.12 (VM), U6.12 (VM), U8.12 (VM)
Other:
- note added: "Battery Charger"
- note added: "Voltage Regulator"
- note removed: "Battery Charger/Monitor"
- note removed: "Voltage Regulators"
- moved on the sheet: C1, C5, C7, C9, D2, R13, R16, R17, R18, U2, U4

Commit message: Layout
Parts:
- removed C7: 4.7uF, Capacitor_SMD:C_0805_2012Metric_Pad1.18x1.45mm_HandSolder, symbol Device:C_Small
- removed C9: 10uF, Capacitor_SMD:C_0805_2012Metric_Pad1.18x1.45mm_HandSolder, symbol Device:C_Small
- removed D2: LED, LED_SMD:LED_0805_2012Metric_Pad1.15x1.40mm_HandSolder, symbol Device:LED
- removed R13: 22Ohms, Resistor_SMD:R_0805_2012Metric_Pad1.20x1.40mm_HandSolder, symbol Device:R
- removed R16, R18: 10KOhms, Resistor_SMD:R_0805_2012Metric_Pad1.20x1.40mm_HandSolder, symbol Device:R
- removed R17: 100KOhms, Resistor_SMD:R_0805_2012Metric_Pad1.20x1.40mm_HandSolder, symbol Device:R
- removed U4: MCP73871, Package_DFN_QFN:QFN-20-1EP_4x4mm_P0.5mm_EP2.5x2.5mm, symbol Battery_Management:MCP73871
- R3: value 2KOhms -> 800Ohms
- SW3: footprint (none) -> Button_Switch_THT:SW_DIP_SPSTx01_Slide_6.7x4.1mm_W7.62mm_P2.54mm_LowProfile
Connections:
- net +5.0V is gone; now on net VBAT_SYS: C13.1, C18.1, C8.1
- net DIRA: now also U9.24 (GPIO47/SPICLK_P/SUBSPICLK_P_DIFF); no longer U9.17 (GPIO9/TOUCH9/ADC1_CH8/FSPIHD/SUBSPIHD)
- net DIRB: now also U9.25 (GPIO48/SPICLK_N/SUBSPICLK_N_DIFF); no longer U9.7 (GPIO7/TOUCH7/ADC1_CH6)
- net DOUT: now also U9.38 (GPIO2/TOUCH2/ADC1_CH1); no longer U9.19 (GPIO11/TOUCH11/ADC2_CH0/FSPID/FSPIIO5/SUBSPID)
- net EN1: now also U9.20 (GPIO12/TOUCH12/ADC2_CH1/FSPICLK/FSPIIO6/SUBSPICLK); no longer U9.4 (GPIO4/TOUCH4/ADC1_CH3)
- net EN2: now also U9.21 (GPIO13/TOUCH13/ADC2_CH2/FSPIQ/FSPIIO7/SUBSPIQ); no longer U9.5 (GPIO5/TOUCH5/ADC1_CH4)
- net EN3: now also U9.22 (GPIO14/TOUCH14/ADC2_CH3/FSPIWP/FSPIDQS/SUBSPIWP); no longer U9.6 (GPIO6/TOUCH6/ADC1_CH5)
- net GND: now also J3.1 (Pin_1); no longer J3.2 (Pin_2)
- net GPIO1_1: now also U9.33 (MTDO/GPIO40/CLK_OUT2); no longer U9.31 (GPIO38/FSPIWP/SUBSPIWP)
- net GPIO1_2: now also U9.34 (MTDI/GPIO41/CLK_OUT1); no longer U9.26 (GPIO45)
- net GPIO1_3: now also U9.35 (MTMS/GPIO42); no longer U9.16 (GPIO46)
- net PD_SCK: now also U9.39 (GPIO1/TOUCH1/ADC1_CH0); no longer U9.20 (GPIO12/TOUCH12/ADC2_CH1/FSPICLK/FSPIIO6/SUBSPICLK)
- net PERC: now also U9.17 (GPIO9/TOUCH9/ADC1_CH8/FSPIHD/SUBSPIHD); no longer U9.38 (GPIO2/TOUCH2/ADC1_CH1)
- net PWMA: now also U9.23 (GPIO21); no longer U9.18 (GPIO10/TOUCH10/ADC1_CH9/FSPICS0/FSPIIO4/SUBSPICS0)
- net PWMB: now also U9.26 (GPIO45); no longer U9.12 (GPIO8/TOUCH8/ADC1_CH7/SUBSPICS1)
- net SCL: now also U9.29 (SPIIO7/GPIO36/FSPICLK/SUBSPICLK); no longer U9.22 (GPIO14/TOUCH14/ADC2_CH3/FSPIWP/FSPIDQS/SUBSPIWP)
- net SDA: now also U9.28 (SPIIO6/GPIO35/FSPID/SUBSPID); no longer U9.21 (GPIO13/TOUCH13/ADC2_CH2/FSPIQ/FSPIIO7/SUBSPIQ)
- net STAT: now also U9.16 (GPIO46); no longer U9.39 (GPIO1/TOUCH1/ADC1_CH0)
- net XSHUT1: now also U9.30 (SPIDQS/GPIO37/FSPIQ/SUBSPIQ); no longer U9.10 (GPIO17/U1TXD/ADC2_CH6)
- net XSHUT2: now also U9.31 (GPIO38/FSPIWP/SUBSPIWP); no longer U9.11 (GPIO18/U1RXD/ADC2_CH7/CLK_OUT3)
- net XSHUT3: now also U9.32 (MTCK/GPIO39/CLK_OUT3/SUBSPICS1); no longer U9.23 (GPIO21)
- net at C14.2, J5.1 (Pin_1), R23.2: now also J3.2 (Pin_2); no longer J3.1 (Pin_1)
- no-connect marks 8 -> 22
Other:
- moved on the sheet: J3

Commit message: Routing
Connections:
- net INA+: now also J7.3 (Pin_3); no longer J7.2 (Pin_2)
- net INA-: now also J7.2 (Pin_2); no longer J7.3 (Pin_3)
- net AOUT1: now reaches U5.2 (AOUT1)
- net AOUT1: now also J1.1 (Pin_1); no longer J1.4 (Pin_4)
- net AOUT2: now reaches U5.4 (AOUT2)
- net AOUT2: now also J1.2 (Pin_2); no longer J1.3 (Pin_3)
- net BOUT2: now reaches U5.5 (BOUT2)
- net BOUT2: now also J1.3 (Pin_3); no longer J1.1 (Pin_1)
- net BOUT1: now reaches U5.7 (BOUT1)
- net BOUT1: now also J1.4 (Pin_4); no longer J1.2 (Pin_2)
- net AOUT1_3: now reaches J9.1 (Pin_1)
- net AOUT1_3: now also U8.2 (AOUT1); no longer U8.5 (BOUT2)
- net AOUT2_3: now reaches J9.2 (Pin_2)
- net AOUT2_3: now also U8.4 (AOUT2); no longer U8.7 (BOUT1)
- net BOUT2_3: now reaches J9.3 (Pin_3)
- net BOUT2_3: now also U8.5 (BOUT2); no longer U8.4 (AOUT2)
- net BOUT1_3: now reaches J9.4 (Pin_4)
- net BOUT1_3: now also U8.7 (BOUT1); no longer U8.2 (AOUT1)
- net AOUT1_2: now reaches J8.1 (Pin_1)
- net AOUT1_2: now also U6.2 (AOUT1); no longer U6.5 (BOUT2)
- net AOUT2_2: now reaches J8.2 (Pin_2)
- net AOUT2_2: now also U6.4 (AOUT2); no longer U6.7 (BOUT1)
- net BOUT2_2: now reaches J8.3 (Pin_3)
- net BOUT2_2: now also U6.5 (BOUT2); no longer U6.4 (AOUT2)
- net BOUT1_2: now reaches J8.4 (Pin_4)
- net BOUT1_2: now also U6.7 (BOUT1); no longer U6.2 (AOUT1)
Other:
- moved on the sheet: J1, J8, J9
