File: Hardware/IR_Sensor/IR_Sensor.kicad_sch (KiCad schematic)
At the start: 31 parts, among them J1 Conn_01x07_Pin, J10 Conn_01x01_Pin, J2 Conn_01x03_Pin, J3 Conn_01x05_Pin, J4 Conn_01x05_Pin, J5 Conn_01x01_Pin, J6 Conn_01x01_Pin, J7 Conn_01x01_Pin, J8 Conn_01x05_Pin, J9 Conn_01x05_Pin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

Commit message: IR Main Board
Parts:
- removed J5, J6: Conn_01x01_Pin, symbol Connector:Conn_01x01_Pin
- added J5: Conn_01x02_Pin, TerminalBlock_Phoenix:TerminalBlock_Phoenix_MKDS-1,5-2_1x02_P5.00mm_Horizontal, symbol Connector:Conn_01x02_Pin
- C1, C2: footprint (none) -> Capacitor_SMD:C_0805_2012Metric_Pad1.18x1.45mm_HandSolder
- J1: footprint (none) -> TerminalBlock_Phoenix:TerminalBlock_Phoenix_MKDS-1,5-7_1x07_P5.00mm_Horizontal
- J2: footprint (none) -> TerminalBlock_Phoenix:TerminalBlock_Phoenix_MKDS-1,5-3_1x03_P5.00mm_Horizontal
- J3, J4: footprint (none) -> TerminalBlock_Phoenix:TerminalBlock_Phoenix_MKDS-1,5-5_1x05_P5.00mm_Horizontal
- R1, R2, R3, R4: footprint (none) -> Resistor_SMD:R_0805_2012Metric_Pad1.20x1.40mm_HandSolder
- U2, U3: footprint Sensor_Distance:ST_VL53L1x -> (none)
Connections:
- net GPIO1_2: now also J5.2 (Pin_2)
- net GPIO1_3: now also J5.1 (Pin_1)
- net SCL: now also J1.2 (Pin_2), J4.2 (Pin_2); no longer J1.3 (Pin_3), J4.3 (Pin_3)
- net SDA: now also J1.3 (Pin_3), J4.3 (Pin_3); no longer J1.2 (Pin_2), J4.2 (Pin_2)
Other:
- note added: "No Place"
- note added: "Sensor Board 2 & 3 -> 1 GPIO1 Bus"
- note removed: "Sensor Board 2 -> 1 GPIO1 Bus"
- note removed: "Sensor Board 3 -> 1 GPIO1 Bus"
- moved on the sheet: J10, J7, J8, J9
