File: Hardware/IR_Sensor/IR_Sensor.kicad_pcb (KiCad board)
At the start: 2 copper layers, 12 parts, among them J1 Conn_01x07_Pin, J2 Conn_01x03_Pin, J3 Conn_01x05_Pin, J4 Conn_01x05_Pin, J5 Conn_01x02_Pin, U1 VL53L0CXV0DH1

Commit message: updated hardware
Routing:
- net GND: track 0.00 -> 7.45 mm, vias 0 -> 21
- net /GPIO1_1: track 34.0 -> 34.6 mm
- added copper zone on B.Cu, net GND
- added copper zone on F.Cu, net GND
Other:
- board outline added: 39 x 48.5 mm
- board text added: "IR Main Board"
- board text added: "NuChef"
- board text added: "Team 62"
